File: portable_display_epass.kicad_pcb (KiCad board)
At the start: 4 copper layers, 58 x 110 mm, 115 parts, among them J1 USB4105-GF-A-060, J2 1S LiPo + NTC, J3 DEBUG POGO, J4 TFT-H035B22WVIST8N20_V3-0, J5 MicroSD, Q1 2N7002, Q2 2N7002, Q3 AO3401A, SW1 UP, SW2 DOWN, SW3 OK, SW4 BACK, SW5 POWER, SW6 FEL, U1 AXP2101, U2 V851s, U3 W25N01GVZEIG, U4 LIS2DW12TR, U5 RV-3028-C7, U6 SN74LVC1G123DCTR, U7 TPS61169DCKR, U8 TPS22918DBVR, U9 USBLC6-2SC6, Y1 24MHz 10ppm

Commit message: feat: initialize EVT1 minboot verification suite and update project validation tools
Parts:
- moved C34 5.83 mm to (15.5, 61.0)
- moved R27 3.00 mm to (42.0, 52.0)
Connections:
- J1 pad A8: (no net) -> unconnected-(J1-SBU1-PadA8)
- J1 pad B8: (no net) -> unconnected-(J1-SBU2-PadB8)
- J4 pad 1: (no net) -> unconnected-(J4-PIN1-Pad1)
- J4 pad 2: (no net) -> unconnected-(J4-PIN2-Pad2)
- J4 pad 3: (no net) -> unconnected-(J4-PIN3-Pad3)
- J4 pad 4: (no net) -> unconnected-(J4-PIN4-Pad4)
- J4 pad 5: (no net) -> unconnected-(J4-PIN5-Pad5)
- U1 pad 10: (no net) -> unconnected-(U1-CPUSLDO-Pad10)
- U1 pad 11: (no net) -> unconnected-(U1-DLDO2_DC4SW-Pad11)
- U1 pad 12: (no net) -> unconnected-(U1-BLDO1-Pad12)
- U1 pad 14: (no net) -> unconnected-(U1-BLDO2-Pad14)
- U1 pad 15: (no net) -> unconnected-(U1-ALDO4-Pad15)
- U1 pad 16: (no net) -> unconnected-(U1-ALDO3-Pad16)
- U1 pad 19: (no net) -> unconnected-(U1-ALDO2-Pad19)
- U1 pad 20: (no net) -> unconnected-(U1-DLDO1_DC1SW-Pad20)
- U1 pad 25: (no net) -> unconnected-(U1-LX2-Pad25)
- U1 pad 26: (no net) -> unconnected-(U1-FB2-Pad26)
- U1 pad 29: PMIC_PWROK -> unconnected-(U1-PWROK-Pad29)
- U1 pad 32: (no net) -> unconnected-(U1-GPIO1_FB5_RTCLDO2-Pad32)
- U1 pad 35: (no net) -> unconnected-(U1-SW-Pad35)
- U2 pad 1: (no net) -> unconnected-(U2-PD18-Pad1)
- U2 pad 18: (no net) -> unconnected-(U2-PE13-Pad18)
- U2 pad 19: (no net) -> unconnected-(U2-PE12-Pad19)
- U2 pad 20: (no net) -> unconnected-(U2-PE11-Pad20)
- U2 pad 27: (no net) -> unconnected-(U2-PE8-Pad27)
- U2 pad 28: (no net) -> unconnected-(U2-PE9-Pad28)
- U2 pad 29: (no net) -> unconnected-(U2-PE3-Pad29)
- U2 pad 32: (no net) -> unconnected-(U2-PE10-Pad32)
- U2 pad 49: (no net) -> unconnected-(U2-LINEOUTP-Pad49)
- U2 pad 52: (no net) -> unconnected-(U2-MICIN1N-Pad52)
- U2 pad 53: (no net) -> unconnected-(U2-MICIN1P-Pad53)
- U2 pad 63: (no net) -> unconnected-(U2-PA11-Pad63)
- U2 pad 64: (no net) -> unconnected-(U2-PA10-Pad64)
- U2 pad 65: (no net) -> unconnected-(U2-PA9-Pad65)
- U2 pad 66: (no net) -> unconnected-(U2-PA8-Pad66)
- U2 pad 67: (no net) -> unconnected-(U2-PA7-Pad67)
- U2 pad 68: (no net) -> unconnected-(U2-PA6-Pad68)
- U2 pad 69: (no net) -> unconnected-(U2-PA5-Pad69)
- U2 pad 70: (no net) -> unconnected-(U2-PA4-Pad70)
- U2 pad 71: (no net) -> unconnected-(U2-PA3-Pad71)
- U2 pad 72: (no net) -> unconnected-(U2-PA2-Pad72)
- U2 pad 73: (no net) -> unconnected-(U2-PA1-Pad73)
- U2 pad 74: (no net) -> unconnected-(U2-PA0-Pad74)
- U2 pad 86: (no net) -> unconnected-(U2-PD7-Pad86)
- U2 pad 87: (no net) -> unconnected-(U2-PD8-Pad87)
- U4 pad 11: (no net) -> unconnected-(U4-INT2-Pad11)
- U4 pad 3: (no net) -> unconnected-(U4-SDO_SA0-Pad3)
- U4 pad 5: (no net) -> unconnected-(U4-NC-Pad5)
- U5 pad 1: (no net) -> unconnected-(U5-CLKOUT-Pad1)
- U8 pad 4: (no net) -> unconnected-(U8-CT-Pad4)
- U8 pad 5: (no net) -> unconnected-(U8-QOD-Pad5)
Routing:
- net ACCEL_INT_N: track 4.11 -> 209.8 mm, vias 2 -> 4
- net PWRON_N: track 1.15 -> 147.7 mm, vias 1 -> 3
- net SD_CLK: track 4.61 -> 142.2 mm
- net RTC_INT_N: track 4.80 -> 131.1 mm, vias 2 -> 3
- net SD_DET: track 4.49 -> 127.4 mm
- net VSYS: track 7.47 -> 124.8 mm, vias 6 -> 12
- net USB_DP: track 5.41 -> 112.8 mm
- net SD_D3: track 4.01 -> 94.6 mm, vias 2 -> 4
- net I2C0_SDA: track 5.42 -> 86.0 mm, vias 3 -> 4
- net NAND_MISO: track 4.05 -> 83.8 mm, vias 2 -> 4
- net SD_CMD: track 4.55 -> 82.5 mm, vias 2 -> 4
- net NAND_MOSI: track 4.61 -> 81.1 mm, vias 2 -> 3
- net SD_D0: track 4.69 -> 80.9 mm, vias 2 -> 3
- net I2C0_SCL: track 6.70 -> 80.6 mm, vias 3 -> 4
- net WAKE_REQ_N: track 1.40 -> 73.1 mm, vias 1 -> 5
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- added copper zone on F.Cu, net 3V3
- added copper zone on F.Cu, net DRAM_1V5
- added copper zone on F.Cu, net SD_3V3
- added copper zone on F.Cu, net VBAT
- added copper zone on F.Cu, net VBUS
- added copper zone on F.Cu, net VSYS

Commit message: gpt6-codex
Routing:
- net USB_DM: track 8.67 -> 100.4 mm, vias 3 -> 4
- net 1V8: track 4.82 -> 94.0 mm, vias 7 -> 13
- net RTC_3V3: track 13.0 -> 102.1 mm, vias 14 -> 17
- net SD_D1: track 4.28 -> 77.1 mm, vias 2 -> 4
- net SD_PWR_EN: track 3.49 -> 74.2 mm, vias 1 -> 8
- net DRAM_1V5: track 10.1 -> 76.5 mm, vias 6 -> 12
- net KEY_DOWN: track 2.50 -> 53.3 mm, vias 0 -> 6
- net 3V3: track 46.3 -> 93.9 mm, vias 32 -> 40
- net STATUS_LED: track 3.62 -> 46.9 mm, vias 1 -> 2
- net PMIC_SDA: track 3.29 -> 33.1 mm, vias 1 -> 6
- net VBUS: track 47.9 -> 75.8 mm, vias 4 -> 6
- net ADC_KEYS: track 22.0 -> 44.3 mm, vias 1 -> 2
- net E907_RX: track 3.15 -> 23.9 mm, vias 1 -> 3
- net STATUS_LED_A: track 0.00 -> 20.0 mm, vias 0 -> 4
- net USB_DP: track 112.8 -> 99.1 mm, vias 3 -> 2
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
Commit message: pcb: experimental U2 relocate + 0.50/0.30 vias (geometry PASS; copper not re-routed)
Automated part move + via ring expand for 0.3 mm drill trial under 2.4" AOD assumption.
Geometry check PASS (radius 26). Tracks not fully reconnected — airwires expected; NOT fab-ready.
Also lands full reference/u2_0p3_fanout_try.patch (no longer stub-only).
Parts:
- moved C37 4.50 mm to (16.4, 61.7)
- moved C12 4.50 mm to (12.6, 52.0)
- moved C13 4.50 mm to (12.6, 60.0)
- moved C34 4.50 mm to (11.2, 62.5)
- moved C15 4.50 mm to (48.3, 61.2)
- moved C18 4.50 mm to (43.2, 69.2)
- moved R27 4.50 mm to (46.3, 50.6)
- moved C35 4.50 mm to (44.5, 56.0)
- moved Y1 4.50 mm to (14.5, 56.0)
- moved C17 4.50 mm to (48.0, 65.0)
- moved C28 4.50 mm to (45.5, 43.1)
- moved C36 4.50 mm to (44.4, 58.9)
- moved C16 4.50 mm to (43.7, 65.6)
- moved C14 4.50 mm to (44.2, 61.7)
- moved D5 4.50 mm to (49.5, 54.7)
