File: 01_power.kicad_sch (KiCad schematic)
At the start: 34 parts, among them J1 USB4105-GF-A-060, J2 1S LiPo + NTC, SW5 POWER, U1 AXP2101, U9 USBLC6-2SC6

Commit message: feat: initialize EVT1 minboot verification suite and update project validation tools
Connections:
- net PMIC_PWROK: no longer names the net of U1.29 (PWROK)
- no-connect marks 14 -> 15
Changed lines of the file:
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@@
 	(global_label "PMIC_BACKUP" (shape passive) (at 320.040 151.130 0) (effects (font (size .8 .8)) (justify left)))
 	(global_label "RTC_3V3" (shape passive) (at 320.040 148.590 0) (effects (font (size .8 .8)) (justify left)))
-	(global_label "PMIC_PWROK" (shape passive) (at 320.040 146.050 0) (effects (font (size .8 .8)) (justify left)))
+	(no_connect (at 320.040 146.050))
 	(global_label "PWRON_N" (shape passive) (at 320.040 143.510 0) (effects (font (size .8 .8)) (justify left)))
 	(global_label "BAT_NTC" (shape passive) (at 320.040 140.970 0) (effects (font (size .8 .8)) (justify left)))
