File: 02_soc_v851s.kicad_sch (KiCad schematic)
At the start: 25 parts, among them J3 DEBUG POGO, SW6 FEL, U2 V851s, U3 W25N01GVZEIG, Y1 24MHz 10ppm

Commit message: feat(display): wire KD024 45-pin MIPI1 on J4; DNP TFT backlight; EL nets TBD
- Replace FPC20 TFT placeholder with Molex 502598-4591 / KD024EGOIN152-01
- IM0/IM1→GND; VCI via U8; VDDIO from 1V8; TE on PD20; DSI lane0 only
- ELVDD/ELVSS/SWIRE nets + probe pads; no invented EL PMIC
- U7 backlight chain DNP; docs/DISPLAY_KD024_NETMAP.md; gates in_progress
- fabrication_released remains false
Connections:
- net LCD_PWM renamed LCD_TE
Changed lines of the file:
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@@
 	(no_connect (at 289.560 195.580))
 	(global_label "LCD_RST" (shape passive) (at 289.560 193.040 180) (effects (font (size .8 .8)) (justify right)))
-	(global_label "LCD_PWM" (shape passive) (at 289.560 190.500 180) (effects (font (size .8 .8)) (justify right)))
+	(global_label "LCD_TE" (shape passive) (at 289.560 190.500 180) (effects (font (size .8 .8)) (justify right)))
 	(global_label "LCD_EN" (shape passive) (at 289.560 187.960 180) (effects (font (size .8 .8)) (justify right)))
 	(global_label "3V3" (shape passive) (at 289.560 185.420 180) (effects (font (size .8 .8)) (justify right)))

Commit message: gpt6-codex
Connections:
- net DSI_D1N: no longer names the net of U2.82 (PD3_DSI_D1N)
- net DSI_D1P: no longer names the net of U2.83 (PD4_DSI_D1P)
- no-connect marks 25 -> 27
Changed lines of the file:
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@@
 	(global_label "DSI_D0N" (shape passive) (at 320.040 107.950 0) (effects (font (size .8 .8)) (justify left)))
 	(global_label "DSI_D0P" (shape passive) (at 320.040 105.410 0) (effects (font (size .8 .8)) (justify left)))
-	(global_label "DSI_D1N" (shape passive) (at 320.040 102.870 0) (effects (font (size .8 .8)) (justify left)))
-	(global_label "DSI_D1P" (shape passive) (at 320.040 100.330 0) (effects (font (size .8 .8)) (justify left)))
+	(no_connect (at 320.040 102.870))
+	(no_connect (at 320.040 100.330))
 	(global_label "DSI_CKN" (shape passive) (at 320.040 97.790 0) (effects (font (size .8 .8)) (justify left)))
 	(global_label "DSI_CKP" (shape passive) (at 320.040 95.250 0) (effects (font (size .8 .8)) (justify left)))
