File: portable_display_epass.kicad_sch (KiCad schematic)
At the start: 0 parts

Commit message: gpt6-codex
Other:
- note added: "EVT1-minboot-r1 - engineering candidate; NOT FOR FABRICATION No radio / no audio / no touch; KD024 AOD firmware pending See docs/ for pin map, power tree and bring-up checklist."
- note removed: "EVT1-minboot-r1 - engineering candidate; NOT FOR FABRICATION No radio / no audio / no touch / no AOD See docs/ for pin map, power tree and bring-up checklist."
Changed lines of the file:
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@@
 		(instances (project "portable_display_epass" (path "/b7613259-1701-5a92-a5a3-2c5d87fd6070" (page "5"))))
 	)
-	(text "EVT1-minboot-r1 - engineering candidate; NOT FOR FABRICATION\nNo radio / no audio / no touch / no AOD\nSee docs/ for pin map, power tree and bring-up checklist." (exclude_from_sim no) (at 25 150 0) (effects (font (size 1.27 1.27)) (justify left top)))
+	(text "EVT1-minboot-r1 - engineering candidate; NOT FOR FABRICATION\nNo radio / no audio / no touch; KD024 AOD firmware pending\nSee docs/ for pin map, power tree and bring-up checklist." (exclude_from_sim no) (at 25 150 0) (effects (font (size 1.27 1.27)) (justify left top)))
 	(sheet_instances (path "/" (page "1")))
 	(embedded_fonts no)
