File: verification/display_completion/checked_project/portable_display_epass.kicad_pcb (KiCad board)
At the start: 4 copper layers, 58 x 110 mm, 124 parts, among them J1 USB4105-GF-A-060, J2 1S LiPo + NTC, J3 DEBUG POGO, J4 KD024EGOIN152-01, J5 MicroSD, Q1 2N7002, Q2 2N7002, Q3 AO3401A, SW1 UP, SW2 DOWN, SW3 OK, SW4 BACK, SW5 POWER, SW6 FEL, U1 AXP2101, U10 TPS65631DPDR, U2 V851s, U3 W25N01GVZEIG, U4 LIS2DW12TR, U5 RV-3028-C7, U6 SN74LVC1G123DCTR, U8 TPS22918DBVR, U9 USBLC6-2SC6, Y1 24MHz 10ppm

Commit message: grok-says-yes
Changed lines of the file:
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@@
 	(segment
 		(start 22.1625 57.4438)
-		(end 26.1 57.4438)
+		(end 24.45 57.4438)
 		(width 0.15)
 		(layer "B.Cu")
@@
 		(layer "B.Cu")
 		(net "SOC_LDO_1V8")
+	)
+	(segment
+		(start 24.45 57.4438)
+		(end 26.1 57.4438)
+		(width 0.15)
+		(layer "B.Cu")
+		(net "SOC_LDO_1V8")
