File: portable-display/hardware/v0_legacy/02_soc_v851s.kicad_sch (KiCad schematic)
At the start: 25 parts, among them J3 DEBUG POGO, SW6 FEL, U2 V851s, U3 W25N01GVZEIG, Y1 24MHz 10ppm

Commit message: refactor: transition to TF-only boot architecture , removing SPI NAND components
Parts:
- removed C22: 100n, Sameat:0402, symbol Sameat:C22_100n
- removed R7: 10k, Sameat:0402, symbol Sameat:R7_10k
- removed R8: 10k, Sameat:0402, symbol Sameat:R8_10k
- removed R9: 10k, Sameat:0402, symbol Sameat:R9_10k
- removed U3: W25N01GVZEIG, Sameat:WSON-8, symbol Sameat:U3_W25N01GVZEIG
Connections:
- net NAND_CLK: no longer names the net of U2.57 (PC0_SPI0_CLK)
- net NAND_CS: no longer names the net of U2.56 (PC1_SPI0_CS)
- net NAND_HOLD: no longer names the net of U2.60 (PC5_SPI0_HOLD)
- net NAND_MISO renamed BOOT1
- net NAND_MOSI renamed BOOT0
- net NAND_WP: no longer names the net of U2.61 (PC4_SPI0_WP)
- no-connect marks 27 -> 31
Other:
- title: 02 V851s / Boot / Storage -> 02 V851s / Boot / TF
