File: portable-display/hardware/v1-WEB6-redesign/split-power-candidate/verification/routing_20260910/work.kicad_pcb (KiCad board)
At the start: 4 copper layers, 38 x 64 mm, 119 parts, among them J1 USB4105-GF-A-060, J2 1S LiPo + NTC, J3 DEBUG POGO, J4 KD024EGOIN152-01, J5 MicroSD, Q1 2N7002, Q2 2N7002, Q3 AO3401A, SW1 UP, SW2 DOWN, SW3 OK, SW4 BACK, SW5 POWER, SW6 FEL, U1 AXP2101, U10 TPS65631DPDR, U2 V851s, U4 LIS2DW12TR, U5 RV-3028-C7, U6 SN74LVC1G123DCTR, U8 TPS22918DBVR, U9 USBLC6-2SC6, Y1 24MHz 10ppm

Commit message: feat: update split-power PCB layout with refined footprints, routing verification data, and updated layout documentation.
Parts:
- moved C6 0.50 mm to (33.8, 52.0)
- moved C7 0.50 mm to (33.8, 53.5)
- moved L2 0.50 mm to (30.4, 52.0)
Routing:
- net USB_CC2: track 66.4 -> 25.7 mm, vias 6 -> 3
- net LCD_EN: track 72.5 -> 51.0 mm
- net VSYS: track 59.2 -> 55.5 mm
- net DRAM_1V5: track 107.1 -> 104.1 mm, vias 6 -> 8
- net CORE_0V93: track 123.9 -> 125.9 mm, vias 12 -> 13
