File: portable-display/hardware/v1-WEB6-redesign/split-power-candidate/01_power.kicad_sch (KiCad schematic)
At the start: 34 parts, among them J1 USB4105-GF-A-060, J2 1S LiPo + NTC, SW5 POWER, U1 AXP2101, U9 USBLC6-2SC6

Commit message: fix: repair USB routing by swapping DP/DM pins on U9 and updating layout files
Connections:
- net USB_DM: now also U9.1 (I/O1), U9.6 (I/O1); no longer U9.3 (I/O2), U9.4 (I/O2)
- net USB_DP: now also U9.3 (I/O2), U9.4 (I/O2); no longer U9.1 (I/O1), U9.6 (I/O1)
Changed lines of the file:
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@@
 	(title_block
 		(title "01 Power / Charger / PMIC")
-		(date "2026-10-01")
-		(rev "WAKE1")
+		(date "2026-10-02")
+		(rev "USB1")
 		(company "Sameat")
 		(comment 1 "Current PCB pin nets; C3036461 factory configuration NOT verified")
@@
 		)
 	)
-	(global_label "USB_DP"
+	(global_label "USB_DM"
 		(shape passive)
 		(at 312.420 49.530 180)
@@
 		)
 	)
-	(global_label "USB_DM"
+	(global_label "USB_DP"
 		(shape passive)
 		(at 312.420 44.450 180)
@@
 		)
 	)
-	(global_label "USB_DM"
+	(global_label "USB_DP"
 		(shape passive)
 		(at 342.900 49.530 0)
@@
 		)
 	)
-	(global_label "USB_DP"
+	(global_label "USB_DM"
 		(shape passive)
 		(at 342.900 44.450 0)

Commit message: fix(pcb): replace D6-D14 with ESDLC5V0LB (C20168172) on dedicated DFN1006-2 land
Parts:
- D13: value PESD4V0 -> ESDLC5V0LB; footprint Sameat:0402 -> Sameat:DFN1006-2; symbol Sameat:D13_PESD4V0 -> Sameat:D13_ESDLC5V0LB; LCSC (none) -> C20168172; MPN PESD4V0Y1BBSF -> ESDLC5V0LB
- D14: value PESD4V0 -> ESDLC5V0LB; footprint Sameat:0402 -> Sameat:DFN1006-2; symbol Sameat:D14_PESD4V0 -> Sameat:D14_ESDLC5V0LB; LCSC (none) -> C20168172; MPN PESD4V0Y1BBSF -> ESDLC5V0LB
Other:
- moved on the sheet: C1, C10, C2, C3, C32, C33, C38, C39, C4, C40, C5, C6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

Commit message: fix(pcb): replace J2 battery connector with 1.0mm SH 3P RA (C7430445) on verified land; reroute VBAT/NTC/VBUS/PMIC_IRQ
Parts:
- J2: footprint Sameat:BAT3 -> Sameat:SH1.0_3P_RA; LCSC C265101 -> C7430445; MPN S3B-PH-SM4-TB(LF)(SN) -> ZX-SH1.0-3PWT
Changed lines of the file:
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@@
 			)
 		)
-		(property "Footprint" "Sameat:BAT3"
+		(property "Footprint" "Sameat:SH1.0_3P_RA"
 			(at 459.740 46.990 0)
 			(effects
@@
 			)
 		)
-		(property "MPN" "S3B-PH-SM4-TB(LF)(SN)"
+		(property "MPN" "ZX-SH1.0-3PWT"
 			(at 459.740 46.990 0)
 			(effects
@@
 			)
 		)
-		(property "LCSC" "C265101"
+		(property "LCSC" "C7430445"
 			(at 459.740 46.990 0)
 			(effects
@@
 			)
 		)
-		(property "Description" ""
+		(property "Description" "1S battery: pin1 VBAT, pin2 NTC, pin3 GND; JST-SH compatible 1.0 mm, 1 A/contact; check battery plug pinout"
 			(at 459.740 46.990 0)
 			(effects

Commit message: feat(power): 0R bring-up isolation links on AXP2101 rails
Connections:
- net 1V8: no longer C10.1, U1.18 (ALDO1)
- net 3V3: no longer C4.1, C5.1, D1.1, L1.2, U1.13 (BLDOIN), U1.17 (ALDOIN), U1.21 (FB1)
- net CORE_0V93: no longer C6.1, C7.1, L2.2, U1.4 (FB3)
- net DRAM_1V5: no longer C8.1, C9.1, L3.2, U1.9 (FB4)
- new net 1V8_PMIC: C10.1, U1.18 (ALDO1)
- new net 3V3_B: D1.1
- new net 3V3_PMIC: C4.1, C5.1, L1.2, U1.13 (BLDOIN), U1.17 (ALDOIN), U1.21 (FB1)
- new net CORE_0V93_PMIC: C6.1, C7.1, L2.2, U1.4 (FB3)
- new net DRAM_1V5_PMIC: C8.1, C9.1, L3.2, U1.9 (FB4)
