File: portable-display/hardware/v1-WEB6-redesign/split-power-candidate/02_soc_v851s.kicad_sch (KiCad schematic)
At the start: 20 parts, among them J3 DEBUG POGO, SW6 FEL, U2 V851s, Y1 24MHz 10ppm

Commit message: fix: resolve screen RESET/TE level matching
Connections:
- net LCD_RST: now also U2.66 (PA8); no longer U2.2 (PD19)
- net LCD_TE: now also U2.65 (PA9); no longer U2.3 (PD20)
Other:
- note added: "DISPLAY GPIO: PA8 (U2.66) -> LCD_RST; PA9 / EINT9 (U2.65) <- LCD_TE. Both use 1V8. R32 10k holds reset LOW at boot. R29 must remain fitted 0R; VDDIO must share the PA supply. Update firmware pin assignments; PD19 / PD20 are now unconnected. See DISPLAY_IO_REPAIR_CN.md."

Commit message: feat: add split power candidate hardware design and wake domain verification reports
Connections:
- net ACCEL_INT_N renamed ACCEL_INT_SOC_N
- net RTC_INT_N renamed RTC_INT_SOC_N
Changed lines of the file:
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@@
 	(title_block
 		(title "02 V851s / Boot / Storage")
-		(date "2026-10-02")
-		(rev "USB1")
+		(date "2026-10-04")
+		(rev "WAKE2")
 		(company "Sameat")
 		(comment 1 "Current PCB pin nets; C3036461 factory configuration NOT verified")
@@
 		)
 	)
-	(global_label "RTC_INT_N"
+	(global_label "RTC_INT_SOC_N"
 		(shape passive)
 		(at 48.260 96.520 180)
@@
 		(at 48.260 83.820)
 	)
-	(global_label "ACCEL_INT_N"
+	(global_label "ACCEL_INT_SOC_N"
 		(shape passive)
 		(at 48.260 81.280 180)

Commit message: fix(sch): regenerate candidate schematic with R33/R34 FEL recovery on PC1
Parts:
- added R33: 1k, Sameat:0402, symbol Sameat:R33_1k
- added R34: 10k, Sameat:0402, symbol Sameat:R34_10k
Connections:
- net 3V3: now also R34.1
- net BOOT0: no longer J3.7 (FEL_PC2), SW6.1 (FEL_PC2), SW6.2 (FEL_PC2)
- net FEL_N: now reaches U2.56 (PC1_SPI0_CS)
- net FEL_N: now also R33.2, R34.2
- new net FEL_KEY_N: J3.7 (FEL_KEY_N), R33.1, SW6.1 (FEL_KEY_N), SW6.2 (FEL_KEY_N)
- no-connect marks 31 -> 30
Other:
- note added: "RECOVERY: hold SW6 before cold power-on. SW6 / J3.7 -> R33 1k -> PC1 / U2.56 (FEL_N). R34 10k pulls FEL_N to switched 3V3. BOOT_SEL[1:0] remains 11 on PC3 / PC2. J3.7: open-drain LOW or release only. BROM tries UART upgrade before USB. See FEL_REPAIR_CN.md."
- moved on the sheet: C12, C13, C14, C15, C16, C17, C18, C19, C20, C21, C34, C35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

Commit message: fix(pcb): add R35 10k LCD_EN pulldown for default-off display power
Parts:
- added R35: 10k, Sameat:0402, symbol Sameat:R35_10k
Connections:
- net GND: now also R35.2
- net LCD_EN: now also R35.1
Other:
- moved on the sheet: C12, C13, C14, C15, C18, C19, C20, C21, C34, C37, R10, R28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

Commit message: feat(j5): swap microSD to in-stock XKTF-0803-0, TPD4E05U06 flow-through ESD, reroute SD bus off Y1
Parts:
- C14: MPN 0402 100n X7R -> CL05B104KO5NNNC
- C34: footprint Sameat:0603 -> Sameat:0402; LCSC (none) -> C12530; MPN (none) -> CL05A225MQ5NSNC
Connections:
- net 3V3: now also C14.2; no longer C14.1
- net GND: now also C14.1; no longer C14.2
Changed lines of the file:
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@@
 			)
 		)
-		(property "MPN" "0402 100n X7R"
+		(property "MPN" "CL05B104KO5NNNC"
 			(at 327.660 163.830 0)
 			(effects
@@
 		)
 	)
+	(global_label "GND"
+		(shape passive)
+		(at 312.420 163.830 180)
+		(effects
+			(font
+				(size .8 .8)
+			)
+			(justify right)
+		)
+	)
 	(global_label "3V3"
-		(shape passive)
-		(at 312.420 163.830 180)
-		(effects
-			(font
-				(size .8 .8)
-			)
-			(justify right)
-		)
-	)
-	(global_label "GND"
 		(shape passive)
 		(at 342.900 163.830 0)
@@
 			)
 		)
-		(property "Footprint" "Sameat:0603"
+		(property "Footprint" "Sameat:0402"
 			(at 327.660 222.250 0)
 			(effects
@@
 			)
 		)
-		(property "MPN" ""
+		(property "MPN" "CL05A225MQ5NSNC"
 			(at 327.660 222.250 0)
 			(effects
@@
 			)
 		)
-		(property "LCSC" ""
+		(property "LCSC" "C12530"
 			(at 327.660 222.250 0)
 			(effects
@@
 			)
 		)
-		(property "Description" "V851SX internal LDOA output bypass"
+		(property "Description" ""
 			(at 327.660 222.250 0)
 			(effects

Commit message: feat(power): 0R bring-up isolation links on AXP2101 rails
Parts:
- added R36: 0R, Sameat:0402, symbol Sameat:R36_0R
- added R37: 0R, Sameat:0402, symbol Sameat:R37_0R
- added R38: 0R, Sameat:0402, symbol Sameat:R38_0R
- added R39: 0R, Sameat:0402, symbol Sameat:R39_0R
- added R40: 0R, Sameat:0402, symbol Sameat:R40_0R
Connections:
- net 1V8: now also R40.2
- net 3V3: now also R39.2; no longer C14.2, U2.5 (VCC33_PF_PD), U2.78 (VCC33_USB)
- net CORE_0V93: now also R36.1
- net DRAM_1V5: now also R37.2
- new net 1V8_PMIC: R40.1
- new net 3V3_B: C14.2, R38.2, U2.5 (VCC33_PF_PD), U2.78 (VCC33_USB)
- new net 3V3_PMIC: R38.1, R39.1
- new net CORE_0V93_PMIC: R36.2
- new net DRAM_1V5_PMIC: R37.1
Other:
- moved on the sheet: C12, C14, C18, C19, C21, C34, C37, R10, R28, R34
