File: portable-display/hardware/v1-WEB6-redesign/split-power-candidate/02_soc_v851s.kicad_sch (KiCad schematic)
At the start: 28 parts, among them J3 DEBUG POGO, SW6 FEL, U2 V851s, Y1 24MHz 10ppm

Commit message: chore(bom): assign LCSC/MPN to 62 parts (JLC basic preferred)
Parts:
- C12, C13: LCSC (none) -> C1549; MPN (none) -> 0402CG180J500NT
- C35: LCSC (none) -> C23630; MPN (none) -> CL10A225KO8NNNC
- C36: LCSC (none) -> C47339; MPN (none) -> CL05A474KP5NNNC
- C37: LCSC (none) -> C1525; MPN (none) -> CL05B104KO5NNNC
- R10, R28: LCSC (none) -> C25744; MPN (none) -> 0402WGF1002TCE
- Y1: LCSC (none) -> C16197264; MPN 24MHz 10ppm 3225 -> XXDBBCNANF-24MHZ
Changed lines of the file:
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@@
 			)
 		)
-		(property "MPN" ""
+		(property "MPN" "CL10A225KO8NNNC"
 			(at 459.740 76.200 0)
 			(effects
@@
 			)
 		)
-		(property "LCSC" ""
+		(property "LCSC" "C23630"
 			(at 459.740 76.200 0)
 			(effects
@@
 			)
 		)
-		(property "MPN" ""
+		(property "MPN" "CL05A474KP5NNNC"
 			(at 327.660 105.410 0)
 			(effects
@@
 			)
 		)
-		(property "LCSC" ""
+		(property "LCSC" "C47339"
 			(at 327.660 105.410 0)
 			(effects
@@
 			)
 		)
-		(property "MPN" ""
+		(property "MPN" "0402CG180J500NT"
 			(at 195.580 134.620 0)
 			(effects
@@
 			)
 		)
-		(property "LCSC" ""
+		(property "LCSC" "C1549"
 			(at 195.580 134.620 0)
 			(effects
@@
 			)
 		)
-		(property "MPN" "24MHz 10ppm 3225"
+		(property "MPN" "XXDBBCNANF-24MHZ"
 			(at 327.660 46.990 0)
 			(effects
@@
 			)
 		)
-		(property "LCSC" ""
+		(property "LCSC" "C16197264"
 			(at 327.660 46.990 0)
 			(effects
@@
 			)
 		)
-		(property "MPN" ""
+		(property "MPN" "0402WGF1002TCE"
 			(at 327.660 163.830 0)
 			(effects
@@
 			)
 		)
-		(property "LCSC" ""
+		(property "LCSC" "C25744"
 			(at 327.660 163.830 0)
 			(effects
@@
 			)
 		)
-		(property "MPN" ""
+		(property "MPN" "0402CG180J500NT"
 			(at 63.500 209.550 0)
 			(effects
@@
 			)
 		)
-		(property "LCSC" ""
+		(property "LCSC" "C1549"
 			(at 63.500 209.550 0)
 			(effects
@@
 			)
 		)
-		(property "MPN" ""
+		(property "MPN" "CL05B104KO5NNNC"
 			(at 195.580 222.250 0)
 			(effects
@@
 			)
 		)
-		(property "LCSC" ""
+		(property "LCSC" "C1525"
 			(at 195.580 222.250 0)
 			(effects
@@
 			)
 		)
-		(property "MPN" ""
+		(property "MPN" "0402WGF1002TCE"
 			(at 195.580 251.460 0)
 			(effects
@@
 			)
 		)
-		(property "LCSC" ""
+		(property "LCSC" "C25744"
 			(at 195.580 251.460 0)
 			(effects

Commit message: `feat(pcb): improve V1 decoupling, test access, and routing`
Parts:
- added TP1: CORE_0V93, Sameat:TestPoint_Pad_D1.0mm, symbol Sameat:TP1_CORE_0V93
- added TP10: GND, Sameat:TestPoint_Pad_D1.0mm, symbol Sameat:TP10_GND
- added TP2: DRAM_1V5, Sameat:TestPoint_Pad_D1.0mm, symbol Sameat:TP2_DRAM_1V5
- added TP3: 1V8, Sameat:TestPoint_Pad_D1.0mm, symbol Sameat:TP3_1V8
Connections:
- net 1V8: now also TP3.1 (TEST)
- net CORE_0V93: now also TP1.1 (TEST)
- net DRAM_1V5: now also TP2.1 (TEST)
- net GND: now also TP10.1 (TEST)
