File: portable-display/hardware/v1-WEB6-redesign/split-power-candidate/03_sensors.kicad_sch (KiCad schematic)
At the start: 25 parts, among them Q1 2N7002, Q2 2N7002, U11 SN74LVC2G17DBVR, U4 LIS2DW12TR, U5 RV-3028-C7, U6 SN74LVC1G123DCTR

Commit message: feat(power): 0R bring-up isolation links on AXP2101 rails
Other:
- moved on the sheet: C57, C59
Changed lines of the file:
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@@
 	)
 	(symbol
-		(lib_id "Sameat:C57_100n")
+		(lib_id "Sameat:C59_100n")
 		(at 63.500 198.120 0)
 		(unit 1)
@@
 		(on_board yes)
 		(dnp no)
-		(property "Reference" "C57"
+		(property "Reference" "C59"
 			(at 63.500 189.040 0)
 			(effects
@@
 			(project "ak_display_38x64_SPLIT_POWER_CANDIDATE"
 				(path "/b7613259-1701-5a92-a5a3-2c5d87fd6070/51072dd9-1bb1-5c78-ad53-b3e9d0a07bc6"
-					(reference "C57")
+					(reference "C59")
 					(unit 1)
 				)
@@
 	)
 	(symbol
-		(lib_id "Sameat:C59_100n")
+		(lib_id "Sameat:C57_100n")
 		(at 195.580 222.250 0)
 		(unit 1)
@@
 		(on_board yes)
 		(dnp no)
-		(property "Reference" "C59"
+		(property "Reference" "C57"
 			(at 195.580 213.170 0)
 			(effects
@@
 			(project "ak_display_38x64_SPLIT_POWER_CANDIDATE"
 				(path "/b7613259-1701-5a92-a5a3-2c5d87fd6070/51072dd9-1bb1-5c78-ad53-b3e9d0a07bc6"
-					(reference "C59")
+					(reference "C57")
 					(unit 1)
 				)

Commit message: feat(pcb): add B-side decoupling for U2 pins 44/37, reroute low-speed GPIO
Parts:
- added C60: 100n, Sameat:0402, symbol Sameat:C60_100n
- added C62: 100n, Sameat:0402, symbol Sameat:C62_100n
Connections:
- net 3V3: now also C60.2
- net GND: now also C60.1, C62.2
- new net 1V8: C62.1
Other:
- moved on the sheet: C57, C59
Changed lines of the file:
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@@
 	)
 	(symbol
-		(lib_id "Sameat:C59_100n")
+		(lib_id "Sameat:C62_100n")
 		(at 63.500 198.120 0)
 		(unit 1)
@@
 		(on_board yes)
 		(dnp no)
-		(property "Reference" "C59"
+		(property "Reference" "C62"
 			(at 63.500 189.040 0)
 			(effects
@@
 			(project "ak_display_38x64_SPLIT_POWER_CANDIDATE"
 				(path "/b7613259-1701-5a92-a5a3-2c5d87fd6070/51072dd9-1bb1-5c78-ad53-b3e9d0a07bc6"
-					(reference "C59")
+					(reference "C62")
 					(unit 1)
 				)
@@
 		)
 	)
+	(global_label "1V8"
+		(shape passive)
+		(at 48.260 198.120 180)
+		(effects
+			(font
+				(size .8 .8)
+			)
+			(justify right)
+		)
+	)
 	(global_label "GND"
 		(shape passive)
-		(at 48.260 198.120 180)
-		(effects
-			(font
-				(size .8 .8)
-			)
-			(justify right)
-		)
-	)
-	(global_label "3V3"
-		(shape passive)
 		(at 78.740 198.120 0)
 		(effects
@@
 	)
 	(symbol
-		(lib_id "Sameat:C57_100n")
+		(lib_id "Sameat:C59_100n")
 		(at 195.580 222.250 0)
 		(unit 1)
@@
 		(on_board yes)
 		(dnp no)
-		(property "Reference" "C57"
+		(property "Reference" "C59"
 			(at 195.580 213.170 0)
 			(effects
@@
 		(property "Description" ""
 			(at 195.580 222.250 0)
+			(effects
+				(font
+					(size 1 1)
+				)
+				(hide yes)
+			)
+		)
+		(pin "1"
+		)
+		(pin "2"
+		)
+		(instances
+			(project "ak_display_38x64_SPLIT_POWER_CANDIDATE"
+				(path "/b7613259-1701-5a92-a5a3-2c5d87fd6070/51072dd9-1bb1-5c78-ad53-b3e9d0a07bc6"
+					(reference "C59")
+					(unit 1)
+				)
+			)
+		)
+	)
+	(global_label "GND"
+		(shape passive)
+		(at 180.340 222.250 180)
+		(effects
+			(font
+				(size .8 .8)
+			)
+			(justify right)
+		)
+	)
+	(global_label "3V3"
+		(shape passive)
+		(at 210.820 222.250 0)
+		(effects
+			(font
+				(size .8 .8)
+			)
+			(justify left)
+		)
+	)
+	(symbol
+		(lib_id "Sameat:C57_100n")
+		(at 327.660 222.250 0)
+		(unit 1)
+		(exclude_from_sim no)
+		(in_bom yes)
+		(on_board yes)
+		(dnp no)
+		(property "Reference" "C57"
+			(at 327.660 213.170 0)
+			(effects
+				(font
+					(size 1 1)
+				)
+			)
+		)
+		(property "Value" "100n"
+			(at 327.660 215.170 0)
+			(effects
+				(font
+					(size 1 1)
+				)
+			)
+		)
+		(property "Footprint" "Sameat:0402"
+			(at 327.660 222.250 0)
+			(effects
+				(font
+					(size 1 1)
+				)
+				(hide yes)
+			)
+		)
+		(property "Datasheet" ""
+			(at 327.660 222.250 0)
+			(effects
+				(font
+					(size 1 1)
+				)
+				(hide yes)
+			)
+		)
+		(property "MPN" "CL05B104KO5NNNC"
+			(at 327.660 222.250 0)
+			(effects
+				(font
+					(size 1 1)
+				)
+				(hide yes)
+			)
+		)
+		(property "LCSC" "C1525"
+			(at 327.660 222.250 0)
+			(effects
+				(font
+					(size 1 1)
+				)
+				(hide yes)
+			)
+		)
+		(property "Description" ""
+			(at 327.660 222.250 0)
 			(effects
 				(font
@@
 	(global_label "GND"
 		(shape passive)
-		(at 180.340 222.250 180)
+		(at 312.420 222.250 180)
 		(effects
 			(font
@@
 	(global_label "3V3"
 		(shape passive)
-		(at 210.820 222.250 0)
-		(effects
-			(font
+		(at 342.900 222.250 0)
+		(effects
+			(font
+				(size .8 .8)
+			)
+			(justify left)
+		)
+	)
+	(symbol
+		(lib_id "Sameat:C60_100n")
+		(at 459.740 222.250 0)
+		(unit 1)
+		(exclude_from_sim no)
+		(in_bom yes)
+		(on_board yes)
+		(dnp no)
+		(property "Reference" "C60"
+			(at 459.740 213.170 0)
+			(effects
+				(font
+					(size 1 1)
+				)
+			)
+		)
+		(property "Value" "100n"
+			(at 459.740 215.170 0)
+			(effects
+				(font
+					(size 1 1)
+				)
+			)
+		)
+		(property "Footprint" "Sameat:0402"
+			(at 459.740 222.250 0)
+			(effects
+				(font
+					(size 1 1)
+				)
+				(hide yes)
+			)
+		)
+		(property "Datasheet" ""
+			(at 459.740 222.250 0)
+			(effects
+				(font
+					(size 1 1)
+				)
+				(hide yes)
+			)
+		)
+		(property "MPN" "CL05B104KO5NNNC"
+			(at 459.740 222.250 0)
+			(effects
+				(font
+					(size 1 1)
+				)
+				(hide yes)
+			)
+		)
+		(property "LCSC" "C1525"
+			(at 459.740 222.250 0)
+			(effects
+				(font
+					(size 1 1)
+				)
+				(hide yes)
+			)
+		)
+		(property "Description" ""
+			(at 459.740 222.250 0)
+			(effects
+				(font
+					(size 1 1)
+				)
+				(hide yes)
+			)
+		)
+		(pin "1"
+		)
+		(pin "2"
+		)
+		(instances
+			(project "ak_display_38x64_SPLIT_POWER_CANDIDATE"
+				(path "/b7613259-1701-5a92-a5a3-2c5d87fd6070/51072dd9-1bb1-5c78-ad53-b3e9d0a07bc6"
+					(reference "C60")
+					(unit 1)
+				)
+			)
+		)
+	)
+	(global_label "GND"
+		(shape passive)
+		(at 444.500 222.250 180)
+		(effects
+			(font
+				(size .8 .8)
+			)
+			(justify right)
+		)
+	)
+	(global_label "3V3"
+		(shape passive)
+		(at 474.980 222.250 0)
+		(effects
+			(font

Commit message: feat(wake): D2/D3 BAT54W C699107, widen SOD-123 land
Parts:
- D2, D3: LCSC (none) -> C699107; MPN (none) -> BAT54W
Changed lines of the file:
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@@
 			)
 		)
-		(property "MPN" ""
+		(property "MPN" "BAT54W"
 			(at 459.740 76.200 0)
 			(effects
@@
 			)
 		)
-		(property "LCSC" ""
+		(property "LCSC" "C699107"
 			(at 459.740 76.200 0)
 			(effects
@@
 			)
 		)
-		(property "MPN" ""
+		(property "MPN" "BAT54W"
 			(at 63.500 139.700 0)
 			(effects
@@
 			)
 		)
-		(property "LCSC" ""
+		(property "LCSC" "C699107"
 			(at 63.500 139.700 0)
 			(effects

Commit message: chore(bom): assign LCSC/MPN to 62 parts (JLC basic preferred)
Parts:
- R11, R13, R14, R17, R18: LCSC (none) -> C25744; MPN (none) -> 0402WGF1002TCE
- R15, R16: LCSC (none) -> C25900; MPN (none) -> 0402WGF4701TCE
- U6: LCSC (none) -> C123302
Changed lines of the file:
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@@
 			)
 		)
-		(property "MPN" ""
+		(property "MPN" "0402WGF1002TCE"
 			(at 63.500 81.280 0)
 			(effects
@@
 			)
 		)
-		(property "LCSC" ""
+		(property "LCSC" "C25744"
 			(at 63.500 81.280 0)
 			(effects
@@
 			)
 		)
-		(property "LCSC" ""
+		(property "LCSC" "C123302"
 			(at 195.580 46.990 0)
 			(effects
@@
 			)
 		)
-		(property "MPN" ""
+		(property "MPN" "0402WGF4701TCE"
 			(at 327.660 105.410 0)
 			(effects
@@
 			)
 		)
-		(property "LCSC" ""
+		(property "LCSC" "C25900"
 			(at 327.660 105.410 0)
 			(effects
@@
 			)
 		)
-		(property "MPN" ""
+		(property "MPN" "0402WGF1002TCE"
 			(at 195.580 163.830 0)
 			(effects
@@
 			)
 		)
-		(property "LCSC" ""
+		(property "LCSC" "C25744"
 			(at 195.580 163.830 0)
 			(effects
@@
 			)
 		)
-		(property "MPN" ""
+		(property "MPN" "0402WGF1002TCE"
 			(at 327.660 163.830 0)
 			(effects
@@
 			)
 		)
-		(property "LCSC" ""
+		(property "LCSC" "C25744"
 			(at 327.660 163.830 0)
 			(effects
@@
 			)
 		)
-		(property "MPN" ""
+		(property "MPN" "0402WGF1002TCE"
 			(at 459.740 163.830 0)
 			(effects
@@
 			)
 		)
-		(property "LCSC" ""
+		(property "LCSC" "C25744"
 			(at 459.740 163.830 0)
 			(effects
@@
 			)
 		)
-		(property "MPN" ""
+		(property "MPN" "0402WGF4701TCE"
 			(at 195.580 193.040 0)
 			(effects
@@
 			)
 		)
-		(property "LCSC" ""
+		(property "LCSC" "C25900"
 			(at 195.580 193.040 0)
 			(effects
@@
 			)
 		)
-		(property "MPN" ""
+		(property "MPN" "0402WGF1002TCE"
 			(at 459.740 193.040 0)
 			(effects
@@
 			)
 		)
-		(property "LCSC" ""
+		(property "LCSC" "C25744"
 			(at 459.740 193.040 0)
 			(effects

Commit message: feat(pcb): B-side 100nF decoupling C56/C58/C61 for U2 CORE pins 13/17/75
Parts:
- added C56: 100n, Sameat:0402, symbol Sameat:C56_100n
- added C58: 100n, Sameat:0402, symbol Sameat:C58_100n
- added C61: 100n, Sameat:0402, symbol Sameat:C61_100n
Connections:
- net GND: now also C56.1, C58.2, C61.1
- new net CORE_0V93: C56.2, C58.1, C61.2
Other:
- moved on the sheet: C57, C59, C60

Commit message: feat(pcb): 3V3_B decoupling C55/C63 for U2-5/78; bring-up, risk and next-rev docs
Parts:
- added C55: 100n, Sameat:0402, symbol Sameat:C55_100n
- added C63: 100n, Sameat:0402, symbol Sameat:C63_100n
Connections:
- net GND: now also C55.2, C63.1
- new net 3V3_B: C55.1, C63.2
Other:
- moved on the sheet: C56, C57, C58, C59, C60, C61
Changed lines of the file:
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@@
 	)
 	(symbol
-		(lib_id "Sameat:C58_100n")
+		(lib_id "Sameat:C55_100n")
 		(at 195.580 222.250 0)
 		(unit 1)
@@
 		(on_board yes)
 		(dnp no)
-		(property "Reference" "C58"
+		(property "Reference" "C55"
 			(at 195.580 213.170 0)
 			(effects
@@
 			(project "ak_display_38x64_SPLIT_POWER_CANDIDATE"
 				(path "/b7613259-1701-5a92-a5a3-2c5d87fd6070/51072dd9-1bb1-5c78-ad53-b3e9d0a07bc6"
-					(reference "C58")
+					(reference "C55")
 					(unit 1)
 				)
@@
 		)
 	)
-	(global_label "CORE_0V93"
+	(global_label "3V3_B"
 		(shape passive)
 		(at 180.340 222.250 180)
@@
 	)
 	(symbol
-		(lib_id "Sameat:C59_100n")
+		(lib_id "Sameat:C58_100n")
 		(at 327.660 222.250 0)
 		(unit 1)
@@
 		(on_board yes)
 		(dnp no)
-		(property "Reference" "C59"
+		(property "Reference" "C58"
 			(at 327.660 213.170 0)
 			(effects
@@
 			(project "ak_display_38x64_SPLIT_POWER_CANDIDATE"
 				(path "/b7613259-1701-5a92-a5a3-2c5d87fd6070/51072dd9-1bb1-5c78-ad53-b3e9d0a07bc6"
-					(reference "C59")
+					(reference "C58")
 					(unit 1)
 				)
@@
 		)
 	)
+	(global_label "CORE_0V93"
+		(shape passive)
+		(at 312.420 222.250 180)
+		(effects
+			(font
+				(size .8 .8)
+			)
+			(justify right)
+		)
+	)
 	(global_label "GND"
 		(shape passive)
-		(at 312.420 222.250 180)
-		(effects
-			(font
-				(size .8 .8)
-			)
-			(justify right)
-		)
-	)
-	(global_label "3V3"
-		(shape passive)
 		(at 342.900 222.250 0)
 		(effects
@@
 	)
 	(symbol
-		(lib_id "Sameat:C56_100n")
+		(lib_id "Sameat:C63_100n")
 		(at 459.740 222.250 0)
 		(unit 1)
@@
 		(on_board yes)
 		(dnp no)
-		(property "Reference" "C56"
+		(property "Reference" "C63"
 			(at 459.740 213.170 0)
 			(effects
@@
 			(project "ak_display_38x64_SPLIT_POWER_CANDIDATE"
 				(path "/b7613259-1701-5a92-a5a3-2c5d87fd6070/51072dd9-1bb1-5c78-ad53-b3e9d0a07bc6"
-					(reference "C56")
+					(reference "C63")
 					(unit 1)
 				)
@@
 		)
 	)
-	(global_label "CORE_0V93"
+	(global_label "3V3_B"
 		(shape passive)
 		(at 474.980 222.250 0)
@@
 	)
 	(symbol
-		(lib_id "Sameat:C61_100n")
+		(lib_id "Sameat:C59_100n")
 		(at 63.500 227.330 0)
 		(unit 1)
@@
 		(on_board yes)
 		(dnp no)
-		(property "Reference" "C61"
+		(property "Reference" "C59"
 			(at 63.500 218.250 0)
 			(effects
@@
 			(project "ak_display_38x64_SPLIT_POWER_CANDIDATE"
 				(path "/b7613259-1701-5a92-a5a3-2c5d87fd6070/51072dd9-1bb1-5c78-ad53-b3e9d0a07bc6"
-					(reference "C61")
+					(reference "C59")
 					(unit 1)
 				)
@@
 		)
 	)
-	(global_label "CORE_0V93"
+	(global_label "3V3"
 		(shape passive)
 		(at 78.740 227.330 0)
@@
 	)
 	(symbol
-		(lib_id "Sameat:C57_100n")
+		(lib_id "Sameat:C56_100n")
 		(at 195.580 251.460 0)
 		(unit 1)
@@
 		(on_board yes)
 		(dnp no)
-		(property "Reference" "C57"
+		(property "Reference" "C56"
 			(at 195.580 242.380 0)
 			(effects
@@
 			(project "ak_display_38x64_SPLIT_POWER_CANDIDATE"
 				(path "/b7613259-1701-5a92-a5a3-2c5d87fd6070/51072dd9-1bb1-5c78-ad53-b3e9d0a07bc6"
-					(reference "C57")
+					(reference "C56")
 					(unit 1)
 				)
@@
 		)
 	)
-	(global_label "3V3"
+	(global_label "CORE_0V93"
 		(shape passive)
 		(at 210.820 251.460 0)
@@
 	)
 	(symbol
-		(lib_id "Sameat:C60_100n")
+		(lib_id "Sameat:C61_100n")
 		(at 327.660 251.460 0)
 		(unit 1)
@@
 		(on_board yes)
 		(dnp no)
-		(property "Reference" "C60"
+		(property "Reference" "C61"
 			(at 327.660 242.380 0)
 			(effects
@@
 		(property "Description" ""
 			(at 327.660 251.460 0)
+			(effects
+				(font
+					(size 1 1)
+				)
+				(hide yes)
+			)
+		)
+		(pin "1"
+		)
+		(pin "2"
+		)
+		(instances
+			(project "ak_display_38x64_SPLIT_POWER_CANDIDATE"
+				(path "/b7613259-1701-5a92-a5a3-2c5d87fd6070/51072dd9-1bb1-5c78-ad53-b3e9d0a07bc6"
+					(reference "C61")
+					(unit 1)
+				)
+			)
+		)
+	)
+	(global_label "GND"
+		(shape passive)
+		(at 312.420 251.460 180)
+		(effects
+			(font
+				(size .8 .8)
+			)
+			(justify right)
+		)
+	)
+	(global_label "CORE_0V93"
+		(shape passive)
+		(at 342.900 251.460 0)
+		(effects
+			(font
+				(size .8 .8)
+			)
+			(justify left)
+		)
+	)
+	(symbol
+		(lib_id "Sameat:C57_100n")
+		(at 459.740 251.460 0)
+		(unit 1)
+		(exclude_from_sim no)
+		(in_bom yes)
+		(on_board yes)
+		(dnp no)
+		(property "Reference" "C57"
+			(at 459.740 242.380 0)
+			(effects
+				(font
+					(size 1 1)
+				)
+			)
+		)
+		(property "Value" "100n"
+			(at 459.740 244.380 0)
+			(effects
+				(font
+					(size 1 1)
+				)
+			)
+		)
+		(property "Footprint" "Sameat:0402"
+			(at 459.740 251.460 0)
+			(effects
+				(font
+					(size 1 1)
+				)
+				(hide yes)
+			)
+		)
+		(property "Datasheet" ""
+			(at 459.740 251.460 0)
+			(effects
+				(font
+					(size 1 1)
+				)
+				(hide yes)
+			)
+		)
+		(property "MPN" "CL05B104KO5NNNC"
+			(at 459.740 251.460 0)
+			(effects
+				(font
+					(size 1 1)
+				)
+				(hide yes)
+			)
+		)
+		(property "LCSC" "C1525"
+			(at 459.740 251.460 0)
+			(effects
+				(font
+					(size 1 1)
+				)
+				(hide yes)
+			)
+		)
+		(property "Description" ""
+			(at 459.740 251.460 0)
+			(effects
+				(font
+					(size 1 1)
+				)
+				(hide yes)
+			)
+		)
+		(pin "1"
+		)
+		(pin "2"
+		)
+		(instances
+			(project "ak_display_38x64_SPLIT_POWER_CANDIDATE"
+				(path "/b7613259-1701-5a92-a5a3-2c5d87fd6070/51072dd9-1bb1-5c78-ad53-b3e9d0a07bc6"
+					(reference "C57")
+					(unit 1)
+				)
+			)
+		)
+	)
+	(global_label "GND"
+		(shape passive)
+		(at 444.500 251.460 180)
+		(effects
+			(font
+				(size .8 .8)
+			)
+			(justify right)
+		)
+	)
+	(global_label "3V3"
+		(shape passive)
+		(at 474.980 251.460 0)
+		(effects
+			(font
+				(size .8 .8)
+			)
+			(justify left)
+		)
+	)
+	(symbol
+		(lib_id "Sameat:C60_100n")
+		(at 63.500 256.540 0)
+		(unit 1)
+		(exclude_from_sim no)
+		(in_bom yes)
+		(on_board yes)
+		(dnp no)
+		(property "Reference" "C60"
+			(at 63.500 247.460 0)
+			(effects
+				(font
+					(size 1 1)
+				)
+			)
+		)
+		(property "Value" "100n"
+			(at 63.500 249.460 0)
+			(effects
+				(font
+					(size 1 1)
+				)
+			)
+		)
+		(property "Footprint" "Sameat:0402"
+			(at 63.500 256.540 0)
+			(effects
+				(font
+					(size 1 1)
+				)
+				(hide yes)
+			)
+		)
+		(property "Datasheet" ""
+			(at 63.500 256.540 0)
+			(effects
+				(font
+					(size 1 1)
+				)
+				(hide yes)
+			)
+		)
+		(property "MPN" "CL05B104KO5NNNC"
+			(at 63.500 256.540 0)
+			(effects
+				(font
+					(size 1 1)
+				)
+				(hide yes)
+			)
+		)
+		(property "LCSC" "C1525"
+			(at 63.500 256.540 0)
+			(effects
+				(font
+					(size 1 1)
+				)
+				(hide yes)
+			)
+		)
+		(property "Description" ""
+			(at 63.500 256.540 0)
 			(effects
 				(font
@@
 	(global_label "GND"
 		(shape passive)
-		(at 312.420 251.460 180)
+		(at 48.260 256.540 180)
 		(effects
 			(font
@@
 	(global_label "3V3"
 		(shape passive)
-		(at 342.900 251.460 0)
-		(effects
-			(font
+		(at 78.740 256.540 0)
+		(effects
+			(font

Commit message: `feat(pcb): improve V1 decoupling, test access, and routing`
Parts:
- added C64: 100n, Sameat:0402, symbol Sameat:C64_100n
- added TP4: RTC_3V3, Sameat:TestPoint_Pad_D1.0mm, symbol Sameat:TP4_RTC_3V3
Connections:
- net 3V3: now also C64.2
- net GND: now also C64.1
- net RTC_3V3: now also TP4.1 (TEST)
Changed lines of the file:
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@@
 	(title_block
 		(title "03 Always-on Sensors / Wake")
-		(date "2026-10-05")
+		(date "2026-10-18")
 		(rev "FEL1")
 		(company "Sameat")
@@
 	)
 	(symbol
+		(lib_id "Sameat:TP4_RTC_3V3")
+		(at 327.660 280.670 0)
+		(unit 1)
+		(exclude_from_sim no)
+		(in_bom no)
+		(on_board yes)
+		(dnp no)
+		(property "Reference" "TP4"
+			(at 327.660 271.590 0)
+			(effects
+				(font
+					(size 1 1)
+				)
+			)
+		)
+		(property "Value" "RTC_3V3"
+			(at 327.660 273.590 0)
+			(effects
+				(font
+					(size 1 1)
+				)
+			)
+		)
+		(property "Footprint" "Sameat:TestPoint_Pad_D1.0mm"
+			(at 327.660 280.670 0)
+			(effects
+				(font
+					(size 1 1)
+				)
+				(hide yes)
+			)
+		)
+		(property "Datasheet" ""
+			(at 327.660 280.670 0)
+			(effects
+				(font
+					(size 1 1)
+				)
+				(hide yes)
+			)
+		)
+		(property "MPN" ""
+			(at 327.660 280.670 0)
+			(effects
+				(font
+					(size 1 1)
+				)
+				(hide yes)
+			)
+		)
+		(property "LCSC" ""
+			(at 327.660 280.670 0)
+			(effects
+				(font
+					(size 1 1)
+				)
+				(hide yes)
+			)
+		)
+		(property "Description" "Bare probe pad; no purchased or assembled part"
+			(at 327.660 280.670 0)
+			(effects
+				(font
+					(size 1 1)
+				)
+				(hide yes)
+			)
+		)
+		(pin "1"
+		)
+		(instances
+			(project "ak_display_38x64_SPLIT_POWER_CANDIDATE"
+				(path "/b7613259-1701-5a92-a5a3-2c5d87fd6070/51072dd9-1bb1-5c78-ad53-b3e9d0a07bc6"
+					(reference "TP4")
+					(unit 1)
+				)
+			)
+		)
+	)
+	(global_label "RTC_3V3"
+		(shape passive)
+		(at 312.420 280.670 180)
+		(effects
+			(font
+				(size .8 .8)
+			)
+			(justify right)
+		)
+	)
+	(symbol
 		(lib_id "Sameat:C60_100n")
 		(at 63.500 256.540 0)
@@
 		(effects
 			(font
+				(size .8 .8)
+			)
+			(justify left)
+		)
+	)
+	(symbol
+		(lib_id "Sameat:C64_100n")
+		(at 195.580 280.670 0)
+		(unit 1)
+		(exclude_from_sim no)
+		(in_bom yes)
+		(on_board yes)
+		(dnp no)
+		(property "Reference" "C64"
+			(at 195.580 271.590 0)
+			(effects
+				(font
+					(size 1 1)
+				)
+			)
+		)
+		(property "Value" "100n"
+			(at 195.580 273.590 0)
+			(effects
+				(font
+					(size 1 1)
+				)
+			)
+		)
+		(property "Footprint" "Sameat:0402"
+			(at 195.580 280.670 0)
+			(effects
+				(font
+					(size 1 1)
+				)
+				(hide yes)
+			)
+		)
+		(property "Datasheet" ""
+			(at 195.580 280.670 0)
+			(effects
+				(font
+					(size 1 1)
+				)
+				(hide yes)
+			)
+		)
+		(property "MPN" "CL05B104KO5NNNC"
+			(at 195.580 280.670 0)
+			(effects
+				(font
+					(size 1 1)
+				)
+				(hide yes)
+			)
+		)
+		(property "LCSC" "C1525"
+			(at 195.580 280.670 0)
+			(effects
+				(font
+					(size 1 1)
+				)
+				(hide yes)
+			)
+		)
+		(property "Description" ""
+			(at 195.580 280.670 0)
+			(effects
+				(font
+					(size 1 1)
+				)
+				(hide yes)
+			)
+		)
+		(pin "1"
+		)
+		(pin "2"
+		)
+		(instances
+			(project "ak_display_38x64_SPLIT_POWER_CANDIDATE"
+				(path "/b7613259-1701-5a92-a5a3-2c5d87fd6070/51072dd9-1bb1-5c78-ad53-b3e9d0a07bc6"
+					(reference "C64")
+					(unit 1)
+				)
+			)
+		)
+	)
+	(global_label "GND"
+		(shape passive)
+		(at 180.340 280.670 180)
+		(effects
+			(font
+				(size .8 .8)
+			)
+			(justify right)
+		)
+	)
+	(global_label "3V3"
+		(shape passive)
+		(at 210.820 280.670 0)
+		(effects
+			(font
