File: portable-display/hardware/v1-WEB6-redesign/split-power-candidate/04_interfaces.kicad_sch (KiCad schematic)
At the start: 38 parts, among them J4 KD024EGOIN152-01, J5 MicroSD, Q3 AO3401A, SW1 UP, SW2 DOWN, SW3 OK, SW4 BACK, U10 TPS65631DPDR, U12 TPD4E05U06DQAR, U13 TPD4E05U06DQAR, U8 TPS22918DBVR

Commit message: feat(power): 0R bring-up isolation links on AXP2101 rails
Connections:
- net 3V3: no longer Q3.2 (S)
- new net 3V3_B: Q3.2 (S)
Other:
- moved on the sheet: C46, C47
Changed lines of the file:
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@@
 		)
 	)
-	(global_label "3V3"
+	(global_label "3V3_B"
 		(shape passive)
 		(at 180.340 102.870 180)
@@
 	)
 	(symbol
-		(lib_id "Sameat:C46_10u")
+		(lib_id "Sameat:C47_10u")
 		(at 195.580 281.940 0)
 		(unit 1)
@@
 		(on_board yes)
 		(dnp no)
-		(property "Reference" "C46"
+		(property "Reference" "C47"
 			(at 195.580 272.860 0)
 			(effects
@@
 			(project "ak_display_38x64_SPLIT_POWER_CANDIDATE"
 				(path "/b7613259-1701-5a92-a5a3-2c5d87fd6070/7309f07d-a051-57ea-bb97-60dcbb9d92b6"
-					(reference "C46")
+					(reference "C47")
 					(unit 1)
 				)
@@
 	)
 	(symbol
-		(lib_id "Sameat:C47_10u")
+		(lib_id "Sameat:C46_10u")
 		(at 327.660 281.940 0)
 		(unit 1)
@@
 		(on_board yes)
 		(dnp no)
-		(property "Reference" "C47"
+		(property "Reference" "C46"
 			(at 327.660 272.860 0)
 			(effects
@@
 			(project "ak_display_38x64_SPLIT_POWER_CANDIDATE"
 				(path "/b7613259-1701-5a92-a5a3-2c5d87fd6070/7309f07d-a051-57ea-bb97-60dcbb9d92b6"
-					(reference "C47")
+					(reference "C46")
 					(unit 1)
 				)

Commit message: feat(display): lock J4 to Molex 502598-4593 (C5365339), length-match DSI pairs
Parts:
- J4: LCSC (none) -> C5365339
Changed lines of the file:
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@@
 			)
 		)
-		(property "LCSC" ""
+		(property "LCSC" "C5365339"
 			(at 63.500 71.120 0)
 			(effects
@@
 			)
 		)
-		(property "Description" "Molex 502598-4593; verify -4591 module FPC compatibility; MIPI 1-lane; EL± from U10"
+		(property "Description" "Molex 502598-4593 (LCSC C5365339): 45P 0.3mm BackFlip dual-contact, direct replacement of KD024-recommended 502598-4591 (obsolete); MIPI 1-lane; EL± from U10"
 			(at 63.500 71.120 0)
 			(effects

Commit message: chore(bom): assign LCSC/MPN to 62 parts (JLC basic preferred)
Parts:
- C29: LCSC (none) -> C19666; MPN (none) -> CL10A475KO8NNNC
- C30, C48, C49, C50: LCSC (none) -> C19702; MPN (none) -> CL10A106KP8NNNC
- C31: LCSC (none) -> C15195; MPN (none) -> CL05B103KB5NNNC
- C42, C44: LCSC (none) -> C15849; MPN (none) -> CL10A105KB8NNNC
- C43, C45, C51: LCSC (none) -> C1525; MPN (none) -> CL05B104KO5NNNC
- D5: LCSC (none) -> C2288; MPN 0603 Blue LED -> KT-0603B
- L5, L6: LCSC (none) -> C97018; MPN 4.7uH 1.5A -> WPN201610U4R7MT
- R20, R32: LCSC (none) -> C25744; MPN (none) -> 0402WGF1002TCE
- R21: LCSC (none) -> C25076; MPN (none) -> 0402WGF1000TCE
- R22, R26: LCSC (none) -> C25741; MPN (none) -> 0402WGF1003TCE
- R23, R29: LCSC (none) -> C17168; MPN (none) -> 0402WGF0000TCE
- R24: LCSC (none) -> C25768; MPN (none) -> 0402WGF2202TCE
- R25: LCSC (none) -> C25792; MPN (none) -> 0402WGF4702TCE
- R27: LCSC (none) -> C25879; MPN (none) -> 0402WGF2201TCE
- U8: LCSC (none) -> C131941
Changed lines of the file:
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@@
 			)
 		)
-		(property "MPN" ""
+		(property "MPN" "0402WGF2201TCE"
 			(at 459.740 127.000 0)
 			(effects
@@
 			)
 		)
-		(property "LCSC" ""
+		(property "LCSC" "C25879"
 			(at 459.740 127.000 0)
 			(effects
@@
 			)
 		)
-		(property "MPN" ""
+		(property "MPN" "CL10A105KB8NNNC"
 			(at 195.580 129.540 0)
 			(effects
@@
 			)
 		)
-		(property "LCSC" ""
+		(property "LCSC" "C15849"
 			(at 195.580 129.540 0)
 			(effects
@@
 			)
 		)
-		(property "MPN" ""
+		(property "MPN" "0402WGF0000TCE"
 			(at 327.660 129.540 0)
 			(effects
@@
 			)
 		)
-		(property "LCSC" ""
+		(property "LCSC" "C17168"
 			(at 327.660 129.540 0)
 			(effects
@@
 			)
 		)
-		(property "MPN" ""
+		(property "MPN" "CL05B104KO5NNNC"
 			(at 63.500 147.320 0)
 			(effects
@@
 			)
 		)
-		(property "LCSC" ""
+		(property "LCSC" "C1525"
 			(at 63.500 147.320 0)
 			(effects
@@
 			)
 		)
-		(property "MPN" "4.7uH 1.5A"
+		(property "MPN" "WPN201610U4R7MT"
 			(at 459.740 152.400 0)
 			(effects
@@
 			)
 		)
-		(property "LCSC" ""
+		(property "LCSC" "C97018"
 			(at 459.740 152.400 0)
 			(effects
@@
 			)
 		)
-		(property "MPN" ""
+		(property "MPN" "0402WGF2202TCE"
 			(at 195.580 154.940 0)
 			(effects
@@
 			)
 		)
-		(property "LCSC" ""
+		(property "LCSC" "C25768"
 			(at 195.580 154.940 0)
 			(effects
@@
 			)
 		)
-		(property "MPN" ""
+		(property "MPN" "0402WGF1000TCE"
 			(at 327.660 154.940 0)
 			(effects
@@
 			)
 		)
-		(property "LCSC" ""
+		(property "LCSC" "C25076"
 			(at 327.660 154.940 0)
 			(effects
@@
 			)
 		)
-		(property "MPN" ""
+		(property "MPN" "0402WGF1003TCE"
 			(at 63.500 172.720 0)
 			(effects
@@
 			)
 		)
-		(property "LCSC" ""
+		(property "LCSC" "C25741"
 			(at 63.500 172.720 0)
 			(effects
@@
 			)
 		)
-		(property "MPN" ""
+		(property "MPN" "CL10A106KP8NNNC"
 			(at 459.740 177.800 0)
 			(effects
@@
 			)
 		)
-		(property "LCSC" ""
+		(property "LCSC" "C19702"
 			(at 459.740 177.800 0)
 			(effects
@@
 			)
 		)
-		(property "MPN" ""
+		(property "MPN" "CL05B104KO5NNNC"
 			(at 195.580 180.340 0)
 			(effects
@@
 			)
 		)
-		(property "LCSC" ""
+		(property "LCSC" "C1525"
 			(at 195.580 180.340 0)
 			(effects
@@
 			)
 		)
-		(property "MPN" ""
+		(property "MPN" "CL05B104KO5NNNC"
 			(at 327.660 180.340 0)
 			(effects
@@
 			)
 		)
-		(property "LCSC" ""
+		(property "LCSC" "C1525"
 			(at 327.660 180.340 0)
 			(effects
@@
 			)
 		)
-		(property "MPN" ""
+		(property "MPN" "0402WGF1002TCE"
 			(at 63.500 198.120 0)
 			(effects
@@
 			)
 		)
-		(property "LCSC" ""
+		(property "LCSC" "C25744"
 			(at 63.500 198.120 0)
 			(effects
@@
 			)
 		)
-		(property "MPN" ""
+		(property "MPN" "CL10A475KO8NNNC"
 			(at 459.740 203.200 0)
 			(effects
@@
 			)
 		)
-		(property "LCSC" ""
+		(property "LCSC" "C19666"
 			(at 459.740 203.200 0)
 			(effects
@@
 			)
 		)
-		(property "MPN" "0603 Blue LED"
+		(property "MPN" "KT-0603B"
 			(at 327.660 205.740 0)
 			(effects
@@
 			)
 		)
-		(property "LCSC" ""
+		(property "LCSC" "C2288"
 			(at 327.660 205.740 0)
 			(effects
@@
 			)
 		)
-		(property "MPN" "4.7uH 1.5A"
+		(property "MPN" "WPN201610U4R7MT"
 			(at 63.500 223.520 0)
 			(effects
@@
 			)
 		)
-		(property "LCSC" ""
+		(property "LCSC" "C97018"
 			(at 63.500 223.520 0)
 			(effects
@@
 			)
 		)
-		(property "MPN" ""
+		(property "MPN" "CL05B103KB5NNNC"
 			(at 459.740 228.600 0)
 			(effects
@@
 			)
 		)
-		(property "LCSC" ""
+		(property "LCSC" "C15195"
 			(at 459.740 228.600 0)
 			(effects
@@
 			)
 		)
-		(property "LCSC" ""
+		(property "LCSC" "C131941"
 			(at 195.580 78.740 0)
 			(effects
@@
 			)
 		)
-		(property "MPN" ""
+		(property "MPN" "0402WGF1003TCE"
 			(at 195.580 231.140 0)
 			(effects
@@
 			)
 		)
-		(property "LCSC" ""
+		(property "LCSC" "C25741"
 			(at 195.580 231.140 0)
 			(effects
@@
 			)
 		)
-		(property "MPN" ""
+		(property "MPN" "CL10A106KP8NNNC"
 			(at 327.660 231.140 0)
 			(effects
@@
 			)
 		)
-		(property "LCSC" ""
+		(property "LCSC" "C19702"
 			(at 327.660 231.140 0)
 			(effects
@@
 			)
 		)
-		(property "MPN" ""
+		(property "MPN" "CL10A106KP8NNNC"
 			(at 63.500 248.920 0)
 			(effects
@@
 			)
 		)
-		(property "LCSC" ""
+		(property "LCSC" "C19702"
 			(at 63.500 248.920 0)
 			(effects
@@
 			)
 		)
-		(property "MPN" ""
+		(property "MPN" "0402WGF1002TCE"
 			(at 459.740 254.000 0)
 			(effects
@@
 			)
 		)
-		(property "LCSC" ""
+		(property "LCSC" "C25744"
 			(at 459.740 254.000 0)
 			(effects
@@
 			)
 		)
-		(property "MPN" ""
+		(property "MPN" "0402WGF0000TCE"
 			(at 195.580 256.540 0)
 			(effects
@@
 			)
 		)
-		(property "LCSC" ""
+		(property "LCSC" "C17168"
 			(at 195.580 256.540 0)
 			(effects
@@
 			)
 		)
-		(property "MPN" ""
+		(property "MPN" "CL10A105KB8NNNC"
 			(at 327.660 256.540 0)
 			(effects
@@
 			)
 		)
-		(property "LCSC" ""
+		(property "LCSC" "C15849"
 			(at 327.660 256.540 0)
 			(effects
@@
 			)
 		)
-		(property "MPN" ""
+		(property "MPN" "0402WGF4702TCE"
 			(at 63.500 274.320 0)
 			(effects
@@
 			)
 		)
-		(property "LCSC" ""
+		(property "LCSC" "C25792"
 			(at 63.500 274.320 0)
 			(effects
@@
 			)
 		)
-		(property "MPN" ""
+		(property "MPN" "CL10A106KP8NNNC"
 			(at 459.740 279.400 0)
 			(effects
@@
 			)
 		)
-		(property "LCSC" ""
+		(property "LCSC" "C19702"
 			(at 459.740 279.400 0)
 			(effects

Commit message: `feat(pcb): improve V1 decoupling, test access, and routing`
Parts:
- added TP6: ELVDD, Sameat:TestPoint_Pad_D1.0mm, symbol Sameat:TP6_ELVDD
- added TP7: ELVSS, Sameat:TestPoint_Pad_D1.0mm, symbol Sameat:TP7_ELVSS
Connections:
- net ELVDD: now also TP6.1 (TEST)
- net ELVSS: now also TP7.1 (TEST)
Changed lines of the file:
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@@
 	(title_block
 		(title "04 Display / SD / Buttons")
-		(date "2026-10-05")
+		(date "2026-10-18")
 		(rev "FEL1")
 		(company "Sameat")
@@
 	)
 	(symbol
+		(lib_id "Sameat:TP6_ELVDD")
+		(at 63.500 299.720 0)
+		(unit 1)
+		(exclude_from_sim no)
+		(in_bom no)
+		(on_board yes)
+		(dnp no)
+		(property "Reference" "TP6"
+			(at 63.500 290.640 0)
+			(effects
+				(font
+					(size 1 1)
+				)
+			)
+		)
+		(property "Value" "ELVDD"
+			(at 63.500 292.640 0)
+			(effects
+				(font
+					(size 1 1)
+				)
+			)
+		)
+		(property "Footprint" "Sameat:TestPoint_Pad_D1.0mm"
+			(at 63.500 299.720 0)
+			(effects
+				(font
+					(size 1 1)
+				)
+				(hide yes)
+			)
+		)
+		(property "Datasheet" ""
+			(at 63.500 299.720 0)
+			(effects
+				(font
+					(size 1 1)
+				)
+				(hide yes)
+			)
+		)
+		(property "MPN" ""
+			(at 63.500 299.720 0)
+			(effects
+				(font
+					(size 1 1)
+				)
+				(hide yes)
+			)
+		)
+		(property "LCSC" ""
+			(at 63.500 299.720 0)
+			(effects
+				(font
+					(size 1 1)
+				)
+				(hide yes)
+			)
+		)
+		(property "Description" "Bare probe pad; no purchased or assembled part"
+			(at 63.500 299.720 0)
+			(effects
+				(font
+					(size 1 1)
+				)
+				(hide yes)
+			)
+		)
+		(pin "1"
+		)
+		(instances
+			(project "ak_display_38x64_SPLIT_POWER_CANDIDATE"
+				(path "/b7613259-1701-5a92-a5a3-2c5d87fd6070/7309f07d-a051-57ea-bb97-60dcbb9d92b6"
+					(reference "TP6")
+					(unit 1)
+				)
+			)
+		)
+	)
+	(global_label "ELVDD"
+		(shape passive)
+		(at 48.260 299.720 180)
+		(effects
+			(font
+				(size .8 .8)
+			)
+			(justify right)
+		)
+	)
+	(symbol
 		(lib_id "Sameat:C47_10u")
 		(at 195.580 281.940 0)
@@
 		)
 	)
+	(symbol
+		(lib_id "Sameat:TP7_ELVSS")
+		(at 459.740 304.800 0)
+		(unit 1)
+		(exclude_from_sim no)
+		(in_bom no)
+		(on_board yes)
+		(dnp no)
+		(property "Reference" "TP7"
+			(at 459.740 295.720 0)
+			(effects
+				(font
+					(size 1 1)
+				)
+			)
+		)
+		(property "Value" "ELVSS"
+			(at 459.740 297.720 0)
+			(effects
+				(font
+					(size 1 1)
+				)
+			)
+		)
+		(property "Footprint" "Sameat:TestPoint_Pad_D1.0mm"
+			(at 459.740 304.800 0)
+			(effects
+				(font
+					(size 1 1)
+				)
+				(hide yes)
+			)
+		)
+		(property "Datasheet" ""
+			(at 459.740 304.800 0)
+			(effects
+				(font
+					(size 1 1)
+				)
+				(hide yes)
+			)
+		)
+		(property "MPN" ""
+			(at 459.740 304.800 0)
+			(effects
+				(font
+					(size 1 1)
+				)
+				(hide yes)
+			)
+		)
+		(property "LCSC" ""
+			(at 459.740 304.800 0)
+			(effects
+				(font
+					(size 1 1)
+				)
+				(hide yes)
+			)
+		)
+		(property "Description" "Bare probe pad; no purchased or assembled part"
+			(at 459.740 304.800 0)
+			(effects
+				(font
+					(size 1 1)
+				)
+				(hide yes)
+			)
+		)
+		(pin "1"
+		)
+		(instances
+			(project "ak_display_38x64_SPLIT_POWER_CANDIDATE"
+				(path "/b7613259-1701-5a92-a5a3-2c5d87fd6070/7309f07d-a051-57ea-bb97-60dcbb9d92b6"
+					(reference "TP7")
+					(unit 1)
+				)
+			)
+		)
+	)
+	(global_label "ELVSS"
+		(shape passive)
+		(at 444.500 304.800 180)
+		(effects
+			(font
+				(size .8 .8)
+			)
+			(justify right)
+		)
+	)
